File: 4_Schematics and Boards Layout/4_6_Schematics/MainBoard/RADAR_Main_Board.brd (EAGLE design)
At the start: 260 x 300 mm, 776 parts, among them J1 142-0731-211, J18 142-0731-211, J19 CJT-T-P-HH-ST-TH1, J20 142-0731-211, J21 CJT-T-P-HH-ST-TH1, J22 142-0731-211, J23 142-0731-211, J24 142-0731-211, J25 142-0731-211, J26 142-0731-211, J27 142-0731-211, J28 142-0731-211, J29 142-0731-211, J30 142-0731-211, J31 142-0731-211, J32 142-0731-211, J33 142-0731-211, J34 142-0731-211, J35 142-0731-211, J36 142-0731-211, J37 142-0731-211, J38 142-0731-211, J39 142-0731-211, J40 142-0731-211, J41 142-0731-211, J42 142-0731-211, J43 142-0731-211, J44 142-0731-211, J45 142-0731-211, J46 142-0731-211, J47 142-0731-211, J48 142-0731-211, J49 142-0731-211, J50 142-0731-211, J51 142-0731-211, J52 142-0731-211, J53 142-0731-211, J54 142-0731-211, J55 142-0731-211, U1 AD9484BCPZ-500, U10 ADS7830IPWR, U11 INA241A3IDGKRDGK0008A-MFG, U13 LTC5552IUDBTRMPBF, U14 SZMMSZ5232BT1G, U15 SZMMSZ5232BT1G, U16 EP4RKU+, U17 SZMMSZ5232BT1G, U2 STM32F746ZGT7, U3 AD9708AR, U37 SZMMSZ5232BT1G, U38 SZMMSZ5232BT1G, U39 SZMMSZ5232BT1G, U4 AD8352ACPZ-R7, U40 SZMMSZ5232BT1G, U41 SZMMSZ5232BT1G, U42 XC7A50T-2FTG256I, U43 SZMMSZ5232BT1G, U44 SZMMSZ5232BT1G, U45 SZMMSZ5232BT1G, U46 SZMMSZ5232BT1G, U47 SZMMSZ5232BT1G, U48 SZMMSZ5232BT1G, U49 SZMMSZ5232BT1G, U5 LTC5552IUDBTRMPBF, U50 SZMMSZ5232BT1G, U51 SZMMSZ5232BT1G, U52 SZMMSZ5232BT1G, U53 SZMMSZ5232BT1G, U54 SZMMSZ5232BT1G, U55 SZMMSZ5232BT1G, U56 SZMMSZ5232BT1G, U57 SZMMSZ5232BT1G, U58 SZMMSZ5232BT1G, U59 SZMMSZ5232BT1G, U6 FT601Q-B-T, U60 SZMMSZ5232BT1G, U61 SZMMSZ5232BT1G, U62 SZMMSZ5232BT1G, U63 SZMMSZ5232BT1G, U64 SZMMSZ5232BT1G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

Commit message: removed a short detected by @Mamenace
Routing:
- net M3S_VCTRL: track 658.5 -> 659.7 mm
Changed lines of the file:
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@@
 <setting verticaltext="up"/>
 </settings>
-<grid distance="1" unitdist="mm" unit="mm" style="lines" multiple="1" display="yes" altdistance="0.003125" altunitdist="mic" altunit="mm"/>
+<grid distance="0.05" unitdist="mm" unit="mm" style="lines" multiple="1" display="yes" altdistance="0.003125" altunitdist="mic" altunit="mm"/>
 <layers>
 <layer number="1" name="Top" color="4" fill="1" visible="yes" active="yes"/>
 <layer number="2" name="Route2" color="16" fill="1" visible="no" active="yes"/>
-<layer number="3" name="Route3" color="17" fill="1" visible="yes" active="yes"/>
-<layer number="4" name="Route4" color="18" fill="1" visible="yes" active="yes"/>
+<layer number="3" name="Route3" color="10" fill="1" visible="yes" active="yes"/>
+<layer number="4" name="Route4" color="14" fill="1" visible="yes" active="yes"/>
 <layer number="5" name="Route5" color="19" fill="1" visible="no" active="yes"/>
 <layer number="6" name="Route6" color="25" fill="1" visible="no" active="no"/>
@@
 <layer number="10" name="Route10" color="29" fill="1" visible="no" active="no"/>
 <layer number="11" name="Route11" color="30" fill="1" visible="no" active="no"/>
-<layer number="12" name="Route12" color="23" fill="1" visible="yes" active="yes"/>
+<layer number="12" name="Route12" color="13" fill="1" visible="yes" active="yes"/>
 <layer number="13" name="Route13" color="21" fill="1" visible="no" active="yes"/>
-<layer number="14" name="Route14" color="22" fill="1" visible="yes" active="yes"/>
+<layer number="14" name="Route14" color="11" fill="1" visible="yes" active="yes"/>
 <layer number="15" name="Route15" color="23" fill="1" visible="no" active="yes"/>
 <layer number="16" name="Bottom" color="1" fill="1" visible="yes" active="yes"/>
@@
 <wire x1="210" y1="232.75" x2="212.3213625" y2="235.0713625" width="0.1" layer="12"/>
 <wire x1="212.3213625" y1="235.0713625" x2="229.232915625" y2="235.0713625" width="0.1" layer="12"/>
-<wire x1="229.232915625" y1="235.0713625" x2="230.441921875" y2="236.28036875" width="0.1" layer="12"/>
-<wire x1="230.441921875" y1="236.28036875" x2="236.71963125" y2="236.28036875" width="0.1" layer="12"/>
-<wire x1="236.71963125" y1="236.28036875" x2="238.25" y2="234.75" width="0.1" layer="12"/>
+<wire x1="238.25" y1="234.75" x2="237.55" y2="235.45" width="0.1" layer="12"/>
+<wire x1="237.55" y1="235.45" x2="236.35" y2="235.45" width="0.1" layer="12"/>
+<wire x1="236.35" y1="235.45" x2="234.55" y2="237.25" width="0.1" layer="12"/>
+<wire x1="234.55" y1="237.25" x2="230.5" y2="237.25" width="0.1" layer="12"/>
+<wire x1="230.5" y1="237.25" x2="230.25" y2="237" width="0.1" layer="12"/>
+<wire x1="230.25" y1="237" x2="229.232915625" y2="235.0713625" width="0.1" layer="12"/>
 </signal>
 <signal name="ADC_DCO_P" class="1">
