File: 4_Schematics and Boards Layout/4_6_Schematics/MainBoard/RADAR_Main_Board.brd (EAGLE design)
At the start: 260 x 300 mm, 789 parts, among them IC1 AT93C46A-10SQ-2.7, J1 142-0731-211, J18 142-0731-211, J19 CJT-T-P-HH-ST-TH1, J20 142-0731-211, J21 CJT-T-P-HH-ST-TH1, J22 142-0731-211, J23 142-0731-211, J24 142-0731-211, J25 142-0731-211, J26 142-0731-211, J27 142-0731-211, J28 142-0731-211, J29 142-0731-211, J30 142-0731-211, J31 142-0731-211, J32 142-0731-211, J33 142-0731-211, J34 142-0731-211, J35 142-0731-211, J36 142-0731-211, J37 142-0731-211, J38 142-0731-211, J39 142-0731-211, J40 142-0731-211, J41 142-0731-211, J42 142-0731-211, J43 142-0731-211, J44 142-0731-211, J45 142-0731-211, J46 142-0731-211, J47 142-0731-211, J48 142-0731-211, J49 142-0731-211, J50 142-0731-211, J51 142-0731-211, J52 142-0731-211, J53 142-0731-211, J54 142-0731-211, J55 142-0731-211, U1 AD9484BCPZ-500, U10 ADS7830IPWR, U11 INA241A3IDGKRDGK0008A-MFG, U13 LTC5552IUDBTRMPBF, U14 SZMMSZ5232BT1G, U15 SZMMSZ5232BT1G, U16 EP4RKU+, U17 SZMMSZ5232BT1G, U2 STM32F746ZGT7, U3 AD9708AR, U37 SZMMSZ5232BT1G, U38 SZMMSZ5232BT1G, U39 SZMMSZ5232BT1G, U4 AD8352ACPZ-R7, U40 SZMMSZ5232BT1G, U41 SZMMSZ5232BT1G, U42 XC7A50T-2FTG256I, U43 SZMMSZ5232BT1G, U44 SZMMSZ5232BT1G, U45 SZMMSZ5232BT1G, U46 SZMMSZ5232BT1G, U47 SZMMSZ5232BT1G, U48 SZMMSZ5232BT1G, U49 SZMMSZ5232BT1G, U5 LTC5552IUDBTRMPBF, U50 SZMMSZ5232BT1G, U51 SZMMSZ5232BT1G, U52 SZMMSZ5232BT1G, U53 SZMMSZ5232BT1G, U54 SZMMSZ5232BT1G, U55 SZMMSZ5232BT1G, U56 SZMMSZ5232BT1G, U57 SZMMSZ5232BT1G, U58 SZMMSZ5232BT1G, U59 SZMMSZ5232BT1G, U6 FT2232HQ, U60 SZMMSZ5232BT1G, U61 SZMMSZ5232BT1G, U62 SZMMSZ5232BT1G, U63 SZMMSZ5232BT1G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

Commit message: Add files via upload
Parts:
- moved C102 143.8 mm to (139.8, 212.9)
- moved C104 143.8 mm to (160.1, 223.3)
- moved C106 143.8 mm to (215.9, 212.9)
- moved C118 143.8 mm to (220.6, 152.0)
- moved C121 143.8 mm to (160.3, 147.1)
- moved C126 143.8 mm to (136.2, 205.5)
- moved C129 143.8 mm to (139.5, 206.1)
- moved C130 143.8 mm to (164.8, 203.5)
- moved C138 143.8 mm to (135.0, 202.7)
- moved C150 143.8 mm to (210.4, 228.7)
- moved C151 143.8 mm to (213.9, 228.7)
- moved C162 143.8 mm to (167.2, 128.0)
- moved C166 143.8 mm to (215.2, 205.8)
- moved C167 143.8 mm to (166.2, 158.1)
- moved C168 143.8 mm to (134.1, 125.8)
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Routing:
- net +3V3_FPGA: track 375.5 -> 90.9 mm
- net GND: vias 2711 -> 3279
- added copper zone on layer 1, net GND
Other:
- board text added: "JP17"
- board text added: "JP3"
- board text added: "RX3"
- board text added: "TX3"
