File: 4_Schematics and Boards Layout/4_6_Schematics/MainBoard/RADAR_Main_Board.sch (EAGLE design)
At the start: 776 parts, among them J1 142-0731-211, J18 142-0731-211, J19 CJT-T-P-HH-ST-TH1, J20 142-0731-211, J21 CJT-T-P-HH-ST-TH1, J22 142-0731-211, J23 142-0731-211, J24 142-0731-211, J25 142-0731-211, J26 142-0731-211, J27 142-0731-211, J28 142-0731-211, J29 142-0731-211, J30 142-0731-211, J31 142-0731-211, J32 142-0731-211, J33 142-0731-211, J34 142-0731-211, J35 142-0731-211, J36 142-0731-211, J37 142-0731-211, J38 142-0731-211, J39 142-0731-211, J40 142-0731-211, J41 142-0731-211, J42 142-0731-211, J43 142-0731-211, J44 142-0731-211, J45 142-0731-211, J46 142-0731-211, J47 142-0731-211, J48 142-0731-211, J49 142-0731-211, J50 142-0731-211, J51 142-0731-211, J52 142-0731-211, J53 142-0731-211, J54 142-0731-211, J55 142-0731-211, U1 AD9484BCPZ-500, U10 ADS7830IPWR, U11 INA241A3IDGKRDGK0008A-MFG, U13 LTC5552IUDBTRMPBF, U14 SZMMSZ5232BT1G, U15 SZMMSZ5232BT1G, U16 EP4RKU+, U17 SZMMSZ5232BT1G, U2 STM32F746ZGT7, U3 AD9708AR, U37 SZMMSZ5232BT1G, U38 SZMMSZ5232BT1G, U39 SZMMSZ5232BT1G, U4 AD8352ACPZ-R7, U40 SZMMSZ5232BT1G, U41 SZMMSZ5232BT1G, U42 XC7A50T-2FTG256I, U43 SZMMSZ5232BT1G, U44 SZMMSZ5232BT1G, U45 SZMMSZ5232BT1G, U46 SZMMSZ5232BT1G, U47 SZMMSZ5232BT1G, U48 SZMMSZ5232BT1G, U49 SZMMSZ5232BT1G, U5 LTC5552IUDBTRMPBF, U50 SZMMSZ5232BT1G, U51 SZMMSZ5232BT1G, U52 SZMMSZ5232BT1G, U53 SZMMSZ5232BT1G, U54 SZMMSZ5232BT1G, U55 SZMMSZ5232BT1G, U56 SZMMSZ5232BT1G, U57 SZMMSZ5232BT1G, U58 SZMMSZ5232BT1G, U59 SZMMSZ5232BT1G, U6 FT601Q-B-T, U60 SZMMSZ5232BT1G, U61 SZMMSZ5232BT1G, U62 SZMMSZ5232BT1G, U63 SZMMSZ5232BT1G, U64 SZMMSZ5232BT1G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

Commit message: Add files via upload
Parts:
- added C187: 4.7uF 35V, SparkFun-Capacitors:4.7UF-POLAR-EIA3528-35V-10%(TANT)
- added C188, C189, C190, C192, C193, C194, C195: 0.1uF, eagle-ltspice:CC0201
- added C191: 3.3uF, eagle-ltspice:CC0201
- added IC1: AT93C46A-10SQ-2.7, atmel:AT93C46A-10SQ-2.7
- added L20: BLM15HB121SN1, inductors:BLM15HB121SN1
- added X2: MINI-USB-32005-201, con-cypressindustries:MINI-USB-32005-201
- added Y1: ECS-120-10-36B2-JTN-TR, SparkFun-Clocks:CRYSTAL-12MHZ
- C159: value 22µF -> 0.1uF; device rcl:C-EUC1206 -> eagle-ltspice:CC0201
- C184: value 10µF -> 12pF; device rcl:C-EUC0805 -> eagle-ltspice:CC0201
- C185: value 100nF -> 12pF; device rcl:C-EUC0402 -> eagle-ltspice:CC0201
- C186: value 1nF -> 4.7uF 35V; device rcl:C-EUC0402 -> SparkFun-Capacitors:4.7UF-POLAR-EIA3528-35V-10%(TANT)
- L19: value (none) -> BLM15HB121SN1; device rcl:L-EUL5650M -> inductors:BLM15HB121SN1
- R145, R83, R84: value 33R -> 10k
- R146: value 33R -> 2.2k
- R60: value 33R -> 1k2_1%
- R61: value 33R -> 1k
- U6: value FT601Q-B-T -> FT2232HQ; device My_Library_RADAR:FT601Q-B-T -> My_Library_RADAR:FT2232HQ
Connections:
- removed net +3V3_FT: C184.1, C185.1, C186.1, L19.2
- new net FT2232_USB_D_N: U6A.DM, X2.2
- new net FT2232_USB_D_P: U6A.DP, X2.3
- new net FT_+1V8: C191.2, U6A.VCORE, U6A.VREGOUT, U6B.VCORE, U6B.VCORE_2
- new net FT_CLKOUT: U42G$5.IO_L12N_T1_MRCC_35, U6A.ACBUS5
- new net FT_D0: U42G$5.IO_L22P_T3_35, U6A.ADBUS0
- new net FT_D1: U42G$5.IO_L21P_T3_DQS_35, U6A.ADBUS1
- new net FT_D2: U42G$5.IO_L21N_T3_DQS_35, U6A.ADBUS2
- new net FT_D3: U42G$5.IO_L16N_T2_35, U6A.ADBUS3
- new net FT_D4: U42G$5.IO_L15P_T2_DQS_35, U6A.ADBUS4
- new net FT_D5: U42G$5.IO_L10N_T1_AD15N_35, U6A.ADBUS5
- new net FT_D6: U42G$5.IO_L7P_T1_AD6P_35, U6A.ADBUS6
- new net FT_D7: U42G$5.IO_L9P_T1_DQS_AD7P_35, U6A.ADBUS7
- new net FT_OE#: U42G$5.IO_L1P_T0_AD4P_35, U6A.ACBUS6
- new net FT_RD#: U42G$5.IO_L4N_T0_35, U6A.ACBUS2
- new net FT_RESET#: R61.2, U6A.RESET-
- new net FT_RXF#: U42G$5.IO_L8N_T1_AD14N_35, U6A.ACBUS0
- new net FT_SIWUA: U42G$5.IO_L3P_T0_DQS_AD5P_35, U6A.ACBUS4
- new net FT_TXE#: U42G$5.IO_L8P_T1_AD14P_35, U6A.ACBUS1
- new net FT_WR#: U42G$5.IO_L3N_T0_DQS_AD5N_35, U6A.ACBUS3
- new net N$117: R60.1, U6A.REF
- new net N$118: C184.1, U6A.OSCI, Y1.1
- new net N$119: C185.1, U6A.OSCO, Y1.2
- new net N$120: C186.+, C188.2, L20.1, U6B.VPLL
- new net N$121: C187.+, C189.1, L19.1, U6B.VPHY
- new net N$122: IC1.CS, R145.1, U6A.EECS
- new net N$123: IC1.SK, R84.1, U6A.EECLK
- new net N$124: IC1.DI, R146.1, U6A.EEDATA
- new net N$90: IC1.DO, R146.2, R83.1
- net +3V3_FPGA: now also C159.2, C190.2, C192.2, C193.2, C194.2, C195.2, IC1.VCC, L19.2, L20.2, R145.2, R61.1, R83.2, R84.2, U6B.VCCIO, U6B.VCCIO_2, U6B.VCCIO_3, U6B.VCCIO_4, U6B.VREGIN; no longer C159.1, L19.1
- net GND: now also C159.1, C186.-, C187.-, C188.1, C189.2, C190.1, C191.1, C192.1, C193.1, C194.1, C195.1, IC1.GND, R60.2, U6A.EPAD, U6A.TEST, U6B.AGND, U6B.GND, U6B.GND_2, U6B.GND_3, U6B.GND_4, U6B.GND_5, U6B.GND_6, U6B.GND_7, U6B.GND_8, X2.4, X2.5; no longer C159.2, C186.2
Other:
- moved on the sheet: C159, C184, C185, L19, R145, R146, R60, R61, R83, R84
